Commit message: Enabled robot joints..

File: urdf/mirabb_rev2.xacro (robot description, xacro)
@@ -2,5 +2,5 @@
 <robot name="mirabb_rev2" xmlns:xacro="http://www.ros.org/wiki/xacro">
 <xacro:include filename="$(find mirabb_rev2_description)/urdf/materials.xacro" />
-<!-- <xacro:include filename="$(find mirabb_rev2_description)/urdf/mirabb_rev2.trans" /> -->
+<xacro:include filename="$(find mirabb_rev2_description)/urdf/mirabb_rev2.trans" />
 <xacro:include filename="$(find mirabb_rev2_description)/urdf/gazebo/mirabb_rev2_materials.gazebo" />
 <xacro:include filename="$(find mirabb_rev2_description)/urdf/gazebo/mirabb_rev2_physics.gazebo" />
@@ -450,6 +450,6 @@
   <child link="abb_link_0_1"/>
 </joint>
-<!-- <joint name="joint_abb_1_to_abb_0" type="continuous"> -->
-<joint name="joint_abb_1_to_abb_0" type="fixed">
+<joint name="joint_abb_1_to_abb_0" type="continuous">
+<!-- <joint name="joint_abb_1_to_abb_0" type="fixed"> -->
   <origin xyz="0.0 0.0 0.139" rpy="0 0 0"/>
   <parent link="abb_link_0_1"/>
@@ -458,6 +458,6 @@
   <limit effort="0" lower="-3.141" upper="3.141" velocity="3.054"/>
 </joint>
-<!-- <joint name="joint_abb_2_to_abb_1" type="continuous"> -->
-<joint name="joint_abb_2_to_abb_1" type="fixed">
+<joint name="joint_abb_2_to_abb_1" type="continuous">
+<!-- <joint name="joint_abb_2_to_abb_1" type="fixed"> -->
   <origin xyz="0.175 -0.1225 0.3355" rpy="0 0 0"/>
   <parent link="abb_link_1_1"/>
@@ -466,6 +466,6 @@
   <limit effort="0" lower="-1.570" upper="2.617" velocity="3.054"/>
 </joint>
-<!-- <joint name="joint_abb_3_to_abb_2" type="continuous"> -->
-<joint name="joint_abb_3_to_abb_2" type="fixed">
+<joint name="joint_abb_3_to_abb_2" type="continuous">
+<!-- <joint name="joint_abb_3_to_abb_2" type="fixed"> -->
   <origin xyz="0.0 -0.0267 1.095" rpy="0 0 0"/>
   <parent link="abb_link_2_1"/>
@@ -474,6 +474,6 @@
   <limit effort="0" lower="-3.141" upper="1.308" velocity="3.054"/>
 </joint>
-<!-- <joint name="joint_abb_4_to_abb_3" type="continuous"> -->
-<joint name="joint_abb_4_to_abb_3" type="fixed">
+<joint name="joint_abb_4_to_abb_3" type="continuous">
+<!-- <joint name="joint_abb_4_to_abb_3" type="fixed"> -->
   <origin xyz="0.3401 0.1492 0.175" rpy="0 0 0"/>
   <parent link="abb_link_3_1"/>
@@ -482,6 +482,6 @@
   <limit effort="0" lower="-6.981" upper="6.981" velocity="4.363"/>
 </joint>
-<!-- <joint name="joint_abb_5_to_abb_4" type="continuous"> -->
-<joint name="joint_abb_5_to_abb_4" type="fixed">
+<joint name="joint_abb_5_to_abb_4" type="continuous">
+<!-- <joint name="joint_abb_5_to_abb_4" type="fixed"> -->
   <origin xyz="0.8904 -0.0205 0.0" rpy="0 0 0"/>
   <parent link="abb_link_4_1"/>
@@ -490,6 +490,6 @@
   <limit effort="0" lower="-2.181" upper="2.094" velocity="4.363"/>
 </joint>
-<!-- <joint name="joint_abb_6_to_abb_5" type="continuous"> -->
-<joint name="joint_abb_6_to_abb_5" type="fixed">
+<joint name="joint_abb_6_to_abb_5" type="continuous">
+<!-- <joint name="joint_abb_6_to_abb_5" type="fixed"> -->
   <origin xyz="0.051 0.0205 0.0" rpy="0 0 0"/>
   <parent link="abb_link_5_1"/>

Commit message: fixed laser and robot arm control

File: urdf/mirabb_rev2.xacro (robot description, xacro)
@@ -456,5 +456,6 @@
   <child link="abb_link_1_1"/>
   <axis xyz="-0.0 0.0 1.0"/>
-  <limit effort="0" lower="-3.141" upper="3.141" velocity="3.054"/>
+  <limit effort="100" lower="-3.141" upper="3.141" velocity="10"/>
+  <!-- <limit effort="0" lower="-3.141" upper="3.141" velocity="3.054"/> -->
 </joint>
 <joint name="joint_abb_2_to_abb_1" type="continuous">
@@ -464,5 +465,6 @@
   <child link="abb_link_2_1"/>
   <axis xyz="-0.0 -1.0 0.0"/>
-  <limit effort="0" lower="-1.570" upper="2.617" velocity="3.054"/>
+  <limit effort="100" lower="-1.570" upper="2.617" velocity="10"/>
+  <!-- <limit effort="0" lower="-1.570" upper="2.617" velocity="3.054"/> -->
 </joint>
 <joint name="joint_abb_3_to_abb_2" type="continuous">
@@ -472,5 +474,6 @@
   <child link="abb_link_3_1"/>
   <axis xyz="0.0 1.0 -0.0"/>
-  <limit effort="0" lower="-3.141" upper="1.308" velocity="3.054"/>
+  <limit effort="100" lower="-3.141" upper="1.308" velocity="10"/>
+  <!-- <limit effort="0" lower="-3.141" upper="1.308" velocity="3.054"/> -->
 </joint>
 <joint name="joint_abb_4_to_abb_3" type="continuous">
@@ -480,5 +483,6 @@
   <child link="abb_link_4_1"/>
   <axis xyz="1.0 0.0 0.0"/>
-  <limit effort="0" lower="-6.981" upper="6.981" velocity="4.363"/>
+  <limit effort="100" lower="-6.981" upper="6.981" velocity="10"/>
+  <!-- <limit effort="0" lower="-6.981" upper="6.981" velocity="4.363"/> -->
 </joint>
 <joint name="joint_abb_5_to_abb_4" type="continuous">
@@ -488,5 +492,6 @@
   <child link="abb_link_5_1"/>
   <axis xyz="0.0 1.0 -0.0"/>
-  <limit effort="0" lower="-2.181" upper="2.094" velocity="4.363"/>
+  <limit effort="100" lower="-2.181" upper="2.094" velocity="10"/>
+  <!-- <limit effort="0" lower="-2.181" upper="2.094" velocity="4.363"/> -->
 </joint>
 <joint name="joint_abb_6_to_abb_5" type="continuous">
@@ -496,5 +501,6 @@
   <child link="abb_link_6_1"/>
   <axis xyz="1.0 0.0 0.0"/>
-  <limit effort="0" lower="-6.981" upper="6.981" velocity="6.283"/>
+  <limit effort="100" lower="-6.981" upper="6.981" velocity="10"/>
+  <!-- <limit effort="0" lower="-6.981" upper="6.981" velocity="6.283"/> -->
 </joint>
 <!-- camera link -->
